File: GeigerVFD.kicad_pcb (KiCad board)
At the start: 2 copper layers, 117.3 x 109.7 mm, 74 parts, among them IC1 TLC555, IC2 LM555, J1 Conn_01x02_Male, J2 3.3V, J3 Conn_01x02_Male, J4 Pulse, Q1 BD137, SW1 Rotary_Encoder_Switch, T1 STN0214, T2 2N4401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

Commit message: finalize
Routing:
- net GND: track 435.5 -> 444.9 mm, vias 10 -> 13
- net Net-(U2-Pad28): track 84.2 -> 75.2 mm
- net Net-(U2-Pad30): track 76.8 -> 83.1 mm
- net /P17: track 47.5 -> 49.3 mm
- net /05G: track 50.0 -> 51.6 mm
- net Net-(U2-Pad31): track 77.8 -> 76.3 mm
- net /11G: track 68.6 -> 70.1 mm
- net R: track 28.6 -> 27.3 mm
- net Net-(IC1-Pad3): track 17.0 -> 15.8 mm
- net Net-(SW1-PadS1): track 38.4 -> 39.4 mm
- net Net-(R15-Pad2): track 31.9 -> 31.1 mm
- net Net-(U2-Pad27): track 88.6 -> 89.3 mm
- net /10G: track 65.3 -> 66.0 mm
- net Net-(J3-Pad2): track 12.1 -> 11.5 mm
- net /06G: track 49.1 -> 49.7 mm
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Other:
- net class Default: clearance 0.2 -> 0.254
- net class Power: clearance 0.2 -> 0.254
- rule trace_clearance: 0.2 -> 0.254
- board text added: "2020-05-14 Sec, Ole & iggy"
- board text removed: "2020-05-13"

Commit message: fix MAX6934 connections: Vcc to 3.3V instead of 5V & DIN to MOSI instead of MISO
Parts:
- renumbered U4 to DS1
Connections:
- DS1 pad 22: (no net) -> Net-(DS1-Pad22)
- DS1 pad 23: (no net) -> Net-(DS1-Pad23)
- IC1 pad 5: (no net) -> Net-(IC1-Pad5)
- U2 pad 16: (no net) -> Net-(U2-Pad16)
- U2 pad 17: (no net) -> Net-(U2-Pad17)
- U2 pad 18: (no net) -> Net-(U2-Pad18)
- U2 pad 2: (no net) -> Net-(U2-Pad2)
- U2 pad 21: (no net) -> Net-(U2-Pad21)
- U2 pad 22: (no net) -> Net-(U2-Pad22)
- U2 pad 23: (no net) -> Net-(U2-Pad23)
- U2 pad 24: (no net) -> Net-(U2-Pad24)
- U2 pad 25: (no net) -> Net-(U2-Pad25)
- U2 pad 29: (no net) -> Net-(U2-Pad29)
- U2 pad 3: (no net) -> Net-(U2-Pad3)
- U2 pad 33: (no net) -> Net-(U2-Pad33)
- U2 pad 35: (no net) -> Net-(U2-Pad35)
- U2 pad 36: (no net) -> Net-(U2-Pad36)
- U2 pad 37: (no net) -> Net-(U2-Pad37)
- U2 pad 38: (no net) -> Net-(U2-Pad38)
- U2 pad 4: (no net) -> Net-(U2-Pad4)
- U2 pad 5: (no net) -> Net-(U2-Pad5)
- U2 pad 6: (no net) -> Net-(U2-Pad6)
- U2 pad 8: (no net) -> Net-(U2-Pad8)
- U3 pad 17: (no net) -> Net-(U3-Pad17)
- U3 pad 19: (no net) -> Net-(U3-Pad19)
- U3 pad 2: (no net) -> Net-(U3-Pad2)
- U3 pad 20: (no net) -> Net-(U3-Pad20)
- U3 pad 25: (no net) -> Net-(U3-Pad25)
- U3 pad 28: (no net) -> Net-(U3-Pad28)
- U3 pad 29: (no net) -> Net-(U3-Pad29)
- U3 pad 43: Net-(U2-Pad27) -> Net-(U2-Pad21)
- U3 pad 44: +5V -> +3V3
- U3 pad 6: (no net) -> Net-(U3-Pad6)
Routing:
- net +3V3: track 53.2 -> 147.6 mm, vias 0 -> 1
- net Net-(U2-Pad21): track 0.00 -> 90.4 mm
- net Net-(U2-Pad27): track 89.3 -> 0.00 mm
- net +5V: track 248.0 -> 219.3 mm, vias 6 -> 5
- net GND: track 444.9 -> 440.5 mm
- net /P17: track 49.3 -> 47.5 mm
- net Net-(JP1-Pad3): track 47.3 -> 46.4 mm
Other:
- board text added: "V2 - Sec, Ole & iggy"
- board text removed: "2020-05-14 Sec, Ole & iggy"
